File: pcb/batterycontrol.kicad_sch (KiCad schematic)
At the start: 4 parts, among them SW1 MST22D18G2_125

Commit message: with errors
Connections:
- no-connect marks 0 -> 2
Changed lines of the file:
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@@
 		(color 0 0 0 0)
+	)
+	(no_connect
+		(at 113.03 52.07)
+	)
+	(no_connect
+		(at 113.03 57.15)
 	)
 	(wire
