File: pcb/batterycontrol.kicad_sch (KiCad schematic)
At the start: 4 parts, among them SW1 MST22D18G2_125

Commit message: finished schematic
Connections:
- net LDO_ONOFF: no longer names the net of R10.2, SW1.3
Changed lines of the file:
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@@
-	)
-	(junction
-		(at 113.03 49.53)
-		(diameter 0)
-		(color 0 0 0 0)
 	)
 	(junction
@@
 		)
 	)
-	(wire
-		(pts
-			(xy 113.03 49.53) (xy 116.84 49.53)
-		)
-		(stroke
-			(width 0)
-			(type default)
-		)
-	)
-	(label "ADC_BATTERY"
+	(hierarchical_label "LDO_EN"
+		(shape input)
+		(at 96.52 57.15 180)
+		(effects
+			(font
+				(size 1.27 1.27)
+			)
+			(justify right)
+		)
+	)
+	(hierarchical_label "ADC_BATTERY"
+		(shape input)
 		(at 67.31 55.88 180)
 		(effects
@@
 				(size 1.27 1.27)
 			)
-			(justify right bottom)
-		)
-	)
-	(global_label "LDO_EN"
-		(shape input)
-		(at 96.52 57.15 180)
-		(fields_autoplaced yes)
-		(effects
-			(font
-				(size 1.27 1.27)
-			)
 			(justify right)
-		)
-		(property "Intersheetrefs" "${INTERSHEET_REFS}"
-			(at 86.4591 57.15 0)
-			(effects
-				(font
-					(size 1.27 1.27)
-				)
-				(justify right)
-				(hide yes)
-			)
-		)
-	)
-	(global_label "LDO_ONOFF"
-		(shape bidirectional)
-		(at 116.84 49.53 0)
-		(fields_autoplaced yes)
-		(effects
-			(font
-				(size 1.27 1.27)
-			)
-			(justify left)
-		)
-		(property "Intersheetrefs" "${INTERSHEET_REFS}"
-			(at 131.7014 49.53 0)
-			(effects
-				(font
-					(size 1.27 1.27)
-				)
-				(justify left)
-				(hide yes)
-			)
 		)
 	)
@@
 		(instances
 			(project "Minicopter"
-				(path "/64f47f0f-737f-4ea8-9b68-9c8ed6450afb/345f8b2d-8ca1-45b4-b603-118598e01ed6"
+				(path "/64f47f0f-737f-4ea8-9b68-9c8ed6450afb/a880b9e6-2cc9-406b-acd1-8115b7529151"
 					(reference "#PWR012")
 					(unit 1)
@@
 		(instances
 			(project ""
-				(path "/64f47f0f-737f-4ea8-9b68-9c8ed6450afb/345f8b2d-8ca1-45b4-b603-118598e01ed6"
+				(path "/64f47f0f-737f-4ea8-9b68-9c8ed6450afb/a880b9e6-2cc9-406b-acd1-8115b7529151"
 					(reference "#PWR09")
 					(unit 1)
@@
 		(instances
 			(project ""
-				(path "/64f47f0f-737f-4ea8-9b68-9c8ed6450afb/345f8b2d-8ca1-45b4-b603-118598e01ed6"
+				(path "/64f47f0f-737f-4ea8-9b68-9c8ed6450afb/a880b9e6-2cc9-406b-acd1-8115b7529151"
 					(reference "R9")
 					(unit 1)
@@
 		(instances
 			(project ""
-				(path "/64f47f0f-737f-4ea8-9b68-9c8ed6450afb/345f8b2d-8ca1-45b4-b603-118598e01ed6"
+				(path "/64f47f0f-737f-4ea8-9b68-9c8ed6450afb/a880b9e6-2cc9-406b-acd1-8115b7529151"
 					(reference "#PWR011")
 					(unit 1)
@@
 		(instances
 			(project ""
-				(path "/64f47f0f-737f-4ea8-9b68-9c8ed6450afb/345f8b2d-8ca1-45b4-b603-118598e01ed6"
+				(path "/64f47f0f-737f-4ea8-9b68-9c8ed6450afb/a880b9e6-2cc9-406b-acd1-8115b7529151"
 					(reference "SW1")
 					(unit 1)
@@
 		(instances
 			(project ""
-				(path "/64f47f0f-737f-4ea8-9b68-9c8ed6450afb/345f8b2d-8ca1-45b4-b603-118598e01ed6"
+				(path "/64f47f0f-737f-4ea8-9b68-9c8ed6450afb/a880b9e6-2cc9-406b-acd1-8115b7529151"
 					(reference "#PWR010")
 					(unit 1)
@@
 		(instances
 			(project ""
-				(path "/64f47f0f-737f-4ea8-9b68-9c8ed6450afb/345f8b2d-8ca1-45b4-b603-118598e01ed6"
+				(path "/64f47f0f-737f-4ea8-9b68-9c8ed6450afb/a880b9e6-2cc9-406b-acd1-8115b7529151"
 					(reference "R10")
 					(unit 1)
@@
 		(instances
 			(project ""
-				(path "/64f47f0f-737f-4ea8-9b68-9c8ed6450afb/345f8b2d-8ca1-45b4-b603-118598e01ed6"
+				(path "/64f47f0f-737f-4ea8-9b68-9c8ed6450afb/a880b9e6-2cc9-406b-acd1-8115b7529151"
 					(reference "R8")
 					(unit 1)

Commit message: schematic done
Parts:
- removed SW1: MST22D18G2_125, SlideSwitchSMDTop:SW-SMD_MST22D18G2, symbol MST22D18G2_125:MST22D18G2_125
- added SW1: SS-12D00, SS-12D00:SS12-D00, symbol SS-12D00:SS-12D00
- R10, R8, R9: footprint (none) -> Resistor_SMD:R_0603_1608Metric
Connections:
- net GND: now also SW1.1 (A)
- net LDO_EN: now also SW1.2 (COM)
- net at R10.2: now also SW1.3 (B)
- no-connect marks 2 -> 0
