File: pcb/battery.kicad_sch (KiCad schematic)
At the start: 0 parts

Commit message: battery
Parts:
- added C5: 10uF, symbol Device:C
- added D3, D4: LED, symbol Device:LED
- added J2: Conn_01x02, symbol Connector_Generic:Conn_01x02
- added R5: 1.2K, symbol Device:R
- added R6, R7: 1K, symbol Device:R
- added U2: TP4056-42-ESOP8, Package_SO:SOIC-8-1EP_3.9x4.9mm_P1.27mm_EP2.41x3.3mm_ThermalVias, symbol Battery_Management:TP4056-42-ESOP8
Connections:
- new net: R5.1, U2.2 (PROG)
- new net: R7.1, U2.6 (~{STDBY})
- new net: R6.2, U2.7 (~{CHRG})
- new net: D3.2 (A), R6.1
- new net: D4.2 (A), R7.2
- new net +5V: D3.1 (K), D4.1 (K), U2.4 (V_{CC}), U2.8 (CE)
- new net +BATT: C5.1, J2.1 (Pin_1), U2.5 (BAT)
- new net GND: C5.2, J2.2 (Pin_2), R5.2, U2.1 (TEMP), U2.3 (GND), U2.9 (EPAD)

Commit message: schematic done
Parts:
- C5: footprint (none) -> Capacitor_SMD:C_0603_1608Metric
- D3, D4: footprint (none) -> LED_SMD:LED_0603_1608Metric
- J2: footprint (none) -> Connector_JST:JST_PH_B2B-PH-SM4-TB_1x02-1MP_P2.00mm_Vertical
- R5, R6, R7: footprint (none) -> Resistor_SMD:R_0603_1608Metric
Changed lines of the file:
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@@
 			)
 		)
-		(property "Footprint" ""
+		(property "Footprint" "Resistor_SMD:R_0603_1608Metric"
 			(at 72.39 67.818 90)
 			(effects
@@
 			)
 		)
-		(property "Footprint" ""
+		(property "Footprint" "Connector_JST:JST_PH_B2B-PH-SM4-TB_1x02-1MP_P2.00mm_Vertical"
 			(at 125.73 60.96 0)
 			(effects
@@
 			)
 		)
-		(property "Footprint" ""
+		(property "Footprint" "LED_SMD:LED_0603_1608Metric"
 			(at 63.5 68.58 0)
 			(effects
@@
 			)
 		)
-		(property "Footprint" ""
+		(property "Footprint" "Resistor_SMD:R_0603_1608Metric"
 			(at 72.39 66.802 90)
 			(effects
@@
 			)
 		)
-		(property "Footprint" ""
+		(property "Footprint" "LED_SMD:LED_0603_1608Metric"
 			(at 63.5 66.04 0)
 			(effects
@@
 			)
 		)
-		(property "Footprint" ""
+		(property "Footprint" "Resistor_SMD:R_0603_1608Metric"
 			(at 96.012 73.66 90)
 			(effects
@@
 			)
 		)
-		(property "Footprint" ""
+		(property "Footprint" "Capacitor_SMD:C_0603_1608Metric"
 			(at 112.7252 69.85 0)
 			(effects
