File: pcb/microcontroller.kicad_sch (KiCad schematic)
At the start: 4 parts, among them U3 ESP32-C3-WROOM-02

Commit message: finished schematic
Other:
- moved on the sheet: C12, R15, R18, U3

Commit message: schematic done
Parts:
- C12: footprint (none) -> Capacitor_SMD:C_0603_1608Metric
- R15, R18: footprint (none) -> Resistor_SMD:R_0603_1608Metric
Changed lines of the file:
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@@
 			)
 		)
-		(property "Footprint" ""
+		(property "Footprint" "Resistor_SMD:R_0603_1608Metric"
 			(at 124.968 69.85 90)
 			(effects
@@
 			)
 		)
-		(property "Footprint" ""
+		(property "Footprint" "Resistor_SMD:R_0603_1608Metric"
 			(at 112.522 102.87 90)
 			(effects
@@
 			)
 		)
-		(property "Footprint" ""
+		(property "Footprint" "Capacitor_SMD:C_0603_1608Metric"
 			(at 124.1552 83.82 0)
 			(effects
