File: pcb/motordrivers.kicad_sch (KiCad schematic)
At the start: 20 parts, among them J3 Conn_01x02_Socket, J4 Conn_01x02_Socket, J5 Conn_01x02_Socket, J6 Conn_01x02_Socket, T1 IRLML6344TRPBF, T2 IRLML6344TRPBF, T3 IRLML6344TRPBF, T4 IRLML6344TRPBF

Commit message: finished schematic
Changed lines of the file:
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@@
 		)
 	)
-	(label "MTR2"
+	(hierarchical_label "MTR4"
+		(shape output)
+		(at 209.55 76.2 180)
+		(effects
+			(font
+				(size 1.27 1.27)
+			)
+			(justify right)
+		)
+	)
+	(hierarchical_label "MTR2"
+		(shape output)
 		(at 99.06 76.2 180)
 		(effects
@@
 				(size 1.27 1.27)
 			)
-			(justify right bottom)
-		)
-	)
-	(label "MTR4"
-		(at 209.55 76.2 180)
-		(effects
-			(font
-				(size 1.27 1.27)
-			)
-			(justify right bottom)
-		)
-	)
-	(label "MTR3"
+			(justify right)
+		)
+	)
+	(hierarchical_label "MTR3"
+		(shape output)
 		(at 152.4 76.2 180)
 		(effects
@@
 				(size 1.27 1.27)
 			)
-			(justify right bottom)
-		)
-	)
-	(label "MTR1"
+			(justify right)
+		)
+	)
+	(hierarchical_label "MTR1"
+		(shape output)
 		(at 44.45 77.47 180)
 		(effects
@@
 				(size 1.27 1.27)
 			)
-			(justify right bottom)
+			(justify right)
 		)
 	)
@@
 		(instances
 			(project "Minicopter"
-				(path "/64f47f0f-737f-4ea8-9b68-9c8ed6450afb/ed609819-b5ba-43b4-b1d2-97343d8298dc"
+				(path "/64f47f0f-737f-4ea8-9b68-9c8ed6450afb/da63f7ab-ab66-4122-9e6c-272b8d61763a"
 					(reference "#PWR020")
 					(unit 1)
@@
 		(instances
 			(project "Minicopter"
-				(path "/64f47f0f-737f-4ea8-9b68-9c8ed6450afb/ed609819-b5ba-43b4-b1d2-97343d8298dc"
+				(path "/64f47f0f-737f-4ea8-9b68-9c8ed6450afb/da63f7ab-ab66-4122-9e6c-272b8d61763a"
 					(reference "J6")
 					(unit 1)
@@
 		(instances
 			(project "Minicopter"
-				(path "/64f47f0f-737f-4ea8-9b68-9c8ed6450afb/ed609819-b5ba-43b4-b1d2-97343d8298dc"
+				(path "/64f47f0f-737f-4ea8-9b68-9c8ed6450afb/da63f7ab-ab66-4122-9e6c-272b8d61763a"
 					(reference "T4")
 					(unit 1)
@@
 		(instances
 			(project "Minicopter"
-				(path "/64f47f0f-737f-4ea8-9b68-9c8ed6450afb/ed609819-b5ba-43b4-b1d2-97343d8298dc"
+				(path "/64f47f0f-737f-4ea8-9b68-9c8ed6450afb/da63f7ab-ab66-4122-9e6c-272b8d61763a"
 					(reference "D6")
 					(unit 1)
@@
 		(instances
 			(project ""
-				(path "/64f47f0f-737f-4ea8-9b68-9c8ed6450afb/ed609819-b5ba-43b4-b1d2-97343d8298dc"
+				(path "/64f47f0f-737f-4ea8-9b68-9c8ed6450afb/da63f7ab-ab66-4122-9e6c-272b8d61763a"
 					(reference "T1")
 					(unit 1)
@@
 		(instances
 			(project "Minicopter"
-				(path "/64f47f0f-737f-4ea8-9b68-9c8ed6450afb/ed609819-b5ba-43b4-b1d2-97343d8298dc"
+				(path "/64f47f0f-737f-4ea8-9b68-9c8ed6450afb/da63f7ab-ab66-4122-9e6c-272b8d61763a"
 					(reference "R14")
 					(unit 1)
@@
 		(instances
 			(project "Minicopter"
-				(path "/64f47f0f-737f-4ea8-9b68-9c8ed6450afb/ed609819-b5ba-43b4-b1d2-97343d8298dc"
+				(path "/64f47f0f-737f-4ea8-9b68-9c8ed6450afb/da63f7ab-ab66-4122-9e6c-272b8d61763a"
 					(reference "#PWR024")
 					(unit 1)
@@
 		(instances
 			(project "Minicopter"
-				(path "/64f47f0f-737f-4ea8-9b68-9c8ed6450afb/ed609819-b5ba-43b4-b1d2-97343d8298dc"
+				(path "/64f47f0f-737f-4ea8-9b68-9c8ed6450afb/da63f7ab-ab66-4122-9e6c-272b8d61763a"
 					(reference "#PWR022")
 					(unit 1)
@@
 		(instances
 			(project "Minicopter"
-				(path "/64f47f0f-737f-4ea8-9b68-9c8ed6450afb/ed609819-b5ba-43b4-b1d2-97343d8298dc"
+				(path "/64f47f0f-737f-4ea8-9b68-9c8ed6450afb/da63f7ab-ab66-4122-9e6c-272b8d61763a"
 					(reference "J5")
 					(unit 1)
@@
 		(instances
 			(project ""
-				(path "/64f47f0f-737f-4ea8-9b68-9c8ed6450afb/ed609819-b5ba-43b4-b1d2-97343d8298dc"
+				(path "/64f47f0f-737f-4ea8-9b68-9c8ed6450afb/da63f7ab-ab66-4122-9e6c-272b8d61763a"
 					(reference "#PWR015")
 					(unit 1)
@@
 		(instances
 			(project ""
-				(path "/64f47f0f-737f-4ea8-9b68-9c8ed6450afb/ed609819-b5ba-43b4-b1d2-97343d8298dc"
+				(path "/64f47f0f-737f-4ea8-9b68-9c8ed6450afb/da63f7ab-ab66-4122-9e6c-272b8d61763a"
 					(reference "J3")
 					(unit 1)
@@
 		(instances
 			(project "Minicopter"
-				(path "/64f47f0f-737f-4ea8-9b68-9c8ed6450afb/ed609819-b5ba-43b4-b1d2-97343d8298dc"
+				(path "/64f47f0f-737f-4ea8-9b68-9c8ed6450afb/da63f7ab-ab66-4122-9e6c-272b8d61763a"
 					(reference "#PWR027")
 					(unit 1)
@@
 		(instances
 			(project "Minicopter"
-				(path "/64f47f0f-737f-4ea8-9b68-9c8ed6450afb/ed609819-b5ba-43b4-b1d2-97343d8298dc"
+				(path "/64f47f0f-737f-4ea8-9b68-9c8ed6450afb/da63f7ab-ab66-4122-9e6c-272b8d61763a"
 					(reference "#PWR019")
 					(unit 1)
@@
 		(instances
 			(project "Minicopter"
-				(path "/64f47f0f-737f-4ea8-9b68-9c8ed6450afb/ed609819-b5ba-43b4-b1d2-97343d8298dc"
+				(path "/64f47f0f-737f-4ea8-9b68-9c8ed6450afb/da63f7ab-ab66-4122-9e6c-272b8d61763a"
 					(reference "T2")
 					(unit 1)
@@
 		(instances
 			(project "Minicopter"
-				(path "/64f47f0f-737f-4ea8-9b68-9c8ed6450afb/ed609819-b5ba-43b4-b1d2-97343d8298dc"
+				(path "/64f47f0f-737f-4ea8-9b68-9c8ed6450afb/da63f7ab-ab66-4122-9e6c-272b8d61763a"
 					(reference "#PWR026")
 					(unit 1)
@@
 		(instances
 			(project "Minicopter"
-				(path "/64f47f0f-737f-4ea8-9b68-9c8ed6450afb/ed609819-b5ba-43b4-b1d2-97343d8298dc"
+				(path "/64f47f0f-737f-4ea8-9b68-9c8ed6450afb/da63f7ab-ab66-4122-9e6c-272b8d61763a"
 					(reference "#PWR025")
 					(unit 1)
@@
 		(instances
 			(project "Minicopter"
-				(path "/64f47f0f-737f-4ea8-9b68-9c8ed6450afb/ed609819-b5ba-43b4-b1d2-97343d8298dc"
+				(path "/64f47f0f-737f-4ea8-9b68-9c8ed6450afb/da63f7ab-ab66-4122-9e6c-272b8d61763a"
 					(reference "#PWR023")
 					(unit 1)
@@
 		(instances
 			(project ""
-				(path "/64f47f0f-737f-4ea8-9b68-9c8ed6450afb/ed609819-b5ba-43b4-b1d2-97343d8298dc"
+				(path "/64f47f0f-737f-4ea8-9b68-9c8ed6450afb/da63f7ab-ab66-4122-9e6c-272b8d61763a"
 					(reference "D5")
 					(unit 1)
@@
 		(instances
 			(project "Minicopter"
-				(path "/64f47f0f-737f-4ea8-9b68-9c8ed6450afb/ed609819-b5ba-43b4-b1d2-97343d8298dc"
+				(path "/64f47f0f-737f-4ea8-9b68-9c8ed6450afb/da63f7ab-ab66-4122-9e6c-272b8d61763a"
 					(reference "#PWR021")
 					(unit 1)
@@
 		(instances
 			(project "Minicopter"
-				(path "/64f47f0f-737f-4ea8-9b68-9c8ed6450afb/ed609819-b5ba-43b4-b1d2-97343d8298dc"
+				(path "/64f47f0f-737f-4ea8-9b68-9c8ed6450afb/da63f7ab-ab66-4122-9e6c-272b8d61763a"
 					(reference "C9")
 					(unit 1)
@@
 		(instances
 			(project ""
-				(path "/64f47f0f-737f-4ea8-9b68-9c8ed6450afb/ed609819-b5ba-43b4-b1d2-97343d8298dc"
+				(path "/64f47f0f-737f-4ea8-9b68-9c8ed6450afb/da63f7ab-ab66-4122-9e6c-272b8d61763a"
 					(reference "C8")
 					(unit 1)
@@
 		(instances
 			(project "Minicopter"
-				(path "/64f47f0f-737f-4ea8-9b68-9c8ed6450afb/ed609819-b5ba-43b4-b1d2-97343d8298dc"
+				(path "/64f47f0f-737f-4ea8-9b68-9c8ed6450afb/da63f7ab-ab66-4122-9e6c-272b8d61763a"
 					(reference "D7")
 					(unit 1)
@@
 		(instances
 			(project "Minicopter"
-				(path "/64f47f0f-737f-4ea8-9b68-9c8ed6450afb/ed609819-b5ba-43b4-b1d2-97343d8298dc"
+				(path "/64f47f0f-737f-4ea8-9b68-9c8ed6450afb/da63f7ab-ab66-4122-9e6c-272b8d61763a"
 					(reference "#PWR028")
 					(unit 1)
@@
 		(instances
 			(project ""
-				(path "/64f47f0f-737f-4ea8-9b68-9c8ed6450afb/ed609819-b5ba-43b4-b1d2-97343d8298dc"
+				(path "/64f47f0f-737f-4ea8-9b68-9c8ed6450afb/da63f7ab-ab66-4122-9e6c-272b8d61763a"
 					(reference "#PWR018")
 					(unit 1)
@@
 		(instances
 			(project ""
-				(path "/64f47f0f-737f-4ea8-9b68-9c8ed6450afb/ed609819-b5ba-43b4-b1d2-97343d8298dc"
+				(path "/64f47f0f-737f-4ea8-9b68-9c8ed6450afb/da63f7ab-ab66-4122-9e6c-272b8d61763a"
 					(reference "R11")
 					(unit 1)
@@
 		(instances
 			(project "Minicopter"
-				(path "/64f47f0f-737f-4ea8-9b68-9c8ed6450afb/ed609819-b5ba-43b4-b1d2-97343d8298dc"
+				(path "/64f47f0f-737f-4ea8-9b68-9c8ed6450afb/da63f7ab-ab66-4122-9e6c-272b8d61763a"
 					(reference "J4")
 					(unit 1)
@@
 		(instances
 			(project "Minicopter"
-				(path "/64f47f0f-737f-4ea8-9b68-9c8ed6450afb/ed609819-b5ba-43b4-b1d2-97343d8298dc"
+				(path "/64f47f0f-737f-4ea8-9b68-9c8ed6450afb/da63f7ab-ab66-4122-9e6c-272b8d61763a"
 					(reference "C10")
 					(unit 1)
@@
 		(instances
 			(project "Minicopter"
-				(path "/64f47f0f-737f-4ea8-9b68-9c8ed6450afb/ed609819-b5ba-43b4-b1d2-97343d8298dc"
+				(path "/64f47f0f-737f-4ea8-9b68-9c8ed6450afb/da63f7ab-ab66-4122-9e6c-272b8d61763a"
 					(reference "R13")
 					(unit 1)
@@
 		(instances
 			(project "Minicopter"
-				(path "/64f47f0f-737f-4ea8-9b68-9c8ed6450afb/ed609819-b5ba-43b4-b1d2-97343d8298dc"
+				(path "/64f47f0f-737f-4ea8-9b68-9c8ed6450afb/da63f7ab-ab66-4122-9e6c-272b8d61763a"
 					(reference "D8")
 					(unit 1)
@@
 		(instances
 			(project "Minicopter"
-				(path "/64f47f0f-737f-4ea8-9b68-9c8ed6450afb/ed609819-b5ba-43b4-b1d2-97343d8298dc"
+				(path "/64f47f0f-737f-4ea8-9b68-9c8ed6450afb/da63f7ab-ab66-4122-9e6c-272b8d61763a"
 					(reference "C11")
 					(unit 1)
@@
 		(instances
 			(project "Minicopter"
-				(path "/64f47f0f-737f-4ea8-9b68-9c8ed6450afb/ed609819-b5ba-43b4-b1d2-97343d8298dc"
+				(path "/64f47f0f-737f-4ea8-9b68-9c8ed6450afb/da63f7ab-ab66-4122-9e6c-272b8d61763a"
 					(reference "T3")
 					(unit 1)
@@
 		(instances
 			(project "Minicopter"
-				(path "/64f47f0f-737f-4ea8-9b68-9c8ed6450afb/ed609819-b5ba-43b4-b1d2-97343d8298dc"
+				(path "/64f47f0f-737f-4ea8-9b68-9c8ed6450afb/da63f7ab-ab66-4122-9e6c-272b8d61763a"
 					(reference "R12")
 					(unit 1)

Commit message: schematic done
Parts:
- C10, C11, C8, C9: footprint (none) -> Capacitor_SMD:C_0603_1608Metric
- J3, J4, J5, J6: footprint (none) -> Connector_JST:JST_GH_BM02B-GHS-TBT_1x02-1MP_P1.25mm_Vertical
- R11, R12, R13, R14: footprint (none) -> Resistor_SMD:R_0603_1608Metric
- T1, T2, T3, T4: footprint SI2302DS-T1:SOT95P237X112-3N -> IRLML6344TRPBF:IRLML6344TRPBF
Changed lines of the file:
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@@
 			)
 		)
-		(property "Footprint" ""
+		(property "Footprint" "Connector_JST:JST_GH_BM02B-GHS-TBT_1x02-1MP_P1.25mm_Vertical"
 			(at 227.33 57.15 0)
 			(effects
@@
 			)
 		)
-		(property "Footprint" "SI2302DS-T1:SOT95P237X112-3N"
+		(property "Footprint" "IRLML6344TRPBF:IRLML6344TRPBF"
 			(at 212.09 76.2 0)
 			(effects
@@
 			)
 		)
-		(property "Footprint" "SI2302DS-T1:SOT95P237X112-3N"
+		(property "Footprint" "IRLML6344TRPBF:IRLML6344TRPBF"
 			(at 46.99 77.47 0)
 			(effects
@@
 			)
 		)
-		(property "Footprint" ""
+		(property "Footprint" "Resistor_SMD:R_0603_1608Metric"
 			(at 209.042 81.28 90)
 			(effects
@@
 			)
 		)
-		(property "Footprint" ""
+		(property "Footprint" "Connector_JST:JST_GH_BM02B-GHS-TBT_1x02-1MP_P1.25mm_Vertical"
 			(at 170.18 57.15 0)
 			(effects
@@
 			)
 		)
-		(property "Footprint" ""
+		(property "Footprint" "Connector_JST:JST_GH_BM02B-GHS-TBT_1x02-1MP_P1.25mm_Vertical"
 			(at 62.23 58.42 0)
 			(effects
@@
 			)
 		)
-		(property "Footprint" "SI2302DS-T1:SOT95P237X112-3N"
+		(property "Footprint" "IRLML6344TRPBF:IRLML6344TRPBF"
 			(at 101.6 76.2 0)
 			(effects
@@
 			)
 		)
-		(property "Footprint" ""
+		(property "Footprint" "Capacitor_SMD:C_0603_1608Metric"
 			(at 106.3752 64.77 0)
 			(effects
@@
 			)
 		)
-		(property "Footprint" ""
+		(property "Footprint" "Capacitor_SMD:C_0603_1608Metric"
 			(at 51.7652 66.04 0)
 			(effects
@@
 			)
 		)
-		(property "Footprint" ""
+		(property "Footprint" "Resistor_SMD:R_0603_1608Metric"
 			(at 43.942 82.55 90)
 			(effects
@@
 			)
 		)
-		(property "Footprint" ""
+		(property "Footprint" "Connector_JST:JST_GH_BM02B-GHS-TBT_1x02-1MP_P1.25mm_Vertical"
 			(at 116.84 57.15 0)
 			(effects
@@
 			)
 		)
-		(property "Footprint" ""
+		(property "Footprint" "Capacitor_SMD:C_0603_1608Metric"
 			(at 159.7152 64.77 0)
 			(effects
@@
 			)
 		)
-		(property "Footprint" ""
+		(property "Footprint" "Resistor_SMD:R_0603_1608Metric"
 			(at 151.892 81.28 90)
 			(effects
@@
 			)
 		)
-		(property "Footprint" ""
+		(property "Footprint" "Capacitor_SMD:C_0603_1608Metric"
 			(at 216.8652 64.77 0)
 			(effects
@@
 			)
 		)
-		(property "Footprint" "SI2302DS-T1:SOT95P237X112-3N"
+		(property "Footprint" "IRLML6344TRPBF:IRLML6344TRPBF"
 			(at 154.94 76.2 0)
 			(effects
@@
 			)
 		)
-		(property "Footprint" ""
+		(property "Footprint" "Resistor_SMD:R_0603_1608Metric"
 			(at 98.552 81.28 90)
 			(effects
