File: pcb/sensor.kicad_sch (KiCad schematic)
At the start: 3 parts

Commit message: finished schematic
Changed lines of the file:
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@@
 		)
 	)
-	(global_label "SDA"
+	(hierarchical_label "SDA"
 		(shape bidirectional)
 		(at 55.88 68.58 180)
-		(fields_autoplaced yes)
 		(effects
 			(font
@@
 			(justify right)
 		)
-		(property "Intersheetrefs" "${INTERSHEET_REFS}"
-			(at 48.2154 68.58 0)
-			(effects
-				(font
-					(size 1.27 1.27)
-				)
-				(justify right)
-				(hide yes)
-			)
-		)
-	)
-	(global_label "SCL"
+	)
+	(hierarchical_label "SCL"
 		(shape bidirectional)
 		(at 55.88 66.04 180)
-		(fields_autoplaced yes)
 		(effects
 			(font
@@
 			(justify right)
 		)
-		(property "Intersheetrefs" "${INTERSHEET_REFS}"
-			(at 48.2759 66.04 0)
-			(effects
-				(font
-					(size 1.27 1.27)
-				)
-				(justify right)
-				(hide yes)
-			)
-		)
 	)
 	(symbol
@@
 		(instances
 			(project ""
-				(path "/64f47f0f-737f-4ea8-9b68-9c8ed6450afb/c3ff5dc2-f9f0-4d07-be2e-e8a81e26d923"
+				(path "/64f47f0f-737f-4ea8-9b68-9c8ed6450afb/738662d6-6c41-4f3e-a588-8d054add7828"
 					(reference "U4")
 					(unit 1)
@@
 		(instances
 			(project "Minicopter"
-				(path "/64f47f0f-737f-4ea8-9b68-9c8ed6450afb/c3ff5dc2-f9f0-4d07-be2e-e8a81e26d923"
+				(path "/64f47f0f-737f-4ea8-9b68-9c8ed6450afb/738662d6-6c41-4f3e-a588-8d054add7828"
 					(reference "#PWR016")
 					(unit 1)
@@
 		(instances
 			(project ""
-				(path "/64f47f0f-737f-4ea8-9b68-9c8ed6450afb/c3ff5dc2-f9f0-4d07-be2e-e8a81e26d923"
+				(path "/64f47f0f-737f-4ea8-9b68-9c8ed6450afb/738662d6-6c41-4f3e-a588-8d054add7828"
 					(reference "C6")
 					(unit 1)
@@
 		(instances
 			(project "Minicopter"
-				(path "/64f47f0f-737f-4ea8-9b68-9c8ed6450afb/c3ff5dc2-f9f0-4d07-be2e-e8a81e26d923"
+				(path "/64f47f0f-737f-4ea8-9b68-9c8ed6450afb/738662d6-6c41-4f3e-a588-8d054add7828"
 					(reference "C7")
 					(unit 1)
@@
 		(instances
 			(project "Minicopter"
-				(path "/64f47f0f-737f-4ea8-9b68-9c8ed6450afb/c3ff5dc2-f9f0-4d07-be2e-e8a81e26d923"
+				(path "/64f47f0f-737f-4ea8-9b68-9c8ed6450afb/738662d6-6c41-4f3e-a588-8d054add7828"
 					(reference "#PWR017")
 					(unit 1)
@@
 		(instances
 			(project ""
-				(path "/64f47f0f-737f-4ea8-9b68-9c8ed6450afb/c3ff5dc2-f9f0-4d07-be2e-e8a81e26d923"
+				(path "/64f47f0f-737f-4ea8-9b68-9c8ed6450afb/738662d6-6c41-4f3e-a588-8d054add7828"
 					(reference "#PWR014")
 					(unit 1)
@@
 		(instances
 			(project ""
-				(path "/64f47f0f-737f-4ea8-9b68-9c8ed6450afb/c3ff5dc2-f9f0-4d07-be2e-e8a81e26d923"
+				(path "/64f47f0f-737f-4ea8-9b68-9c8ed6450afb/738662d6-6c41-4f3e-a588-8d054add7828"
 					(reference "#PWR013")
 					(unit 1)

Commit message: schematic done
Parts:
- C6, C7: footprint (none) -> Capacitor_SMD:C_0603_1608Metric
- U4: value ~ -> GY-87_Module; footprint (none) -> GY-87_Module:GY-87_Module
Changed lines of the file:
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@@
-	)
-	(symbol
-		(lib_id "GY-87:GY-87")
-		(at 69.85 67.31 0)
-		(unit 1)
-		(exclude_from_sim no)
-		(in_bom yes)
-		(on_board yes)
-		(dnp no)
-		(property "Reference" "U4"
-			(at 60.198 57.404 0)
-			(effects
-				(font
-					(size 1.27 1.27)
-				)
-				(justify left)
-			)
-		)
-		(property "Value" "~"
-			(at 70.7233 81.28 0)
-			(effects
-				(font
-					(size 1.27 1.27)
-				)
-				(justify left)
-			)
-		)
-		(property "Footprint" ""
-			(at 69.85 67.31 0)
-			(effects
-				(font
-					(size 1.27 1.27)
-				)
-				(hide yes)
-			)
-		)
-		(property "Datasheet" ""
-			(at 69.85 67.31 0)
-			(effects
-				(font
-					(size 1.27 1.27)
-				)
-				(hide yes)
-			)
-		)
-		(property "Description" ""
-			(at 69.85 67.31 0)
-			(effects
-				(font
-					(size 1.27 1.27)
-				)
-				(hide yes)
-			)
-		)
-		(pin "4"
-		)
-		(pin "3"
-		)
-		(pin "7"
-		)
-		(pin "5"
-		)
-		(pin "1"
-		)
-		(pin "6"
-		)
-		(pin "2"
-		)
-		(pin "8"
-		)
-		(instances
-			(project ""
-				(path "/64f47f0f-737f-4ea8-9b68-9c8ed6450afb/738662d6-6c41-4f3e-a588-8d054add7828"
-					(reference "U4")
-					(unit 1)
-				)
-			)
-		)
 	)
 	(symbol
@@
 			)
 		)
-		(property "Footprint" ""
+		(property "Footprint" "Capacitor_SMD:C_0603_1608Metric"
 			(at 89.8652 64.77 0)
 			(effects
@@
 			)
 		)
-		(property "Footprint" ""
+		(property "Footprint" "Capacitor_SMD:C_0603_1608Metric"
 			(at 96.2152 64.77 0)
 			(effects
@@
 					(unit 1)
 				)
+			)
+		)
+	)
+	(symbol
+		(lib_name "GY-87_1")
+		(lib_id "GY-87:GY-87")
+		(at 69.85 67.31 0)
+		(unit 1)
+		(exclude_from_sim no)
+		(in_bom yes)
+		(on_board yes)
+		(dnp no)
+		(fields_autoplaced yes)
+		(property "Reference" "U4"
+			(at 70.7233 80.01 0)
+			(effects
+				(font
+					(size 1.27 1.27)
+				)
+				(justify left)
+			)
+		)
+		(property "Value" "GY-87_Module"
+			(at 70.7233 82.55 0)
+			(effects
+				(font
+					(size 1.27 1.27)
+				)
+				(justify left)
+			)
+		)
+		(property "Footprint" "GY-87_Module:GY-87_Module"
+			(at 69.342 43.942 0)
+			(effects
+				(font
+					(size 1.27 1.27)
+				)
+				(hide yes)
+			)
+		)
+		(property "Datasheet" "kicad-embed://gy-87-10dof-mpu6050-hmc5883l-bmp180-sensor-module.pdf"
+			(at 69.85 41.148 0)
+			(effects
+				(font
+					(size 1.27 1.27)
+				)
+				(hide yes)
+			)
+		)
+		(property "Description" ""
+			(at 69.85 67.31 0)
+			(effects
+				(font
+					(size 1.27 1.27)
+				)
+				(hide yes)
+			)
+		)
+		(pin "8"
+		)
+		(pin "1"
+		)
+		(pin "5"
+		)
+		(pin "6"
+		)
+		(pin "3"
+		)
+		(pin "2"
+		)
+		(pin "7"
+		)
+		(pin "4"
+		)
+		(instances
+			(project ""
+				(path "/64f47f0f-737f-4ea8-9b68-9c8ed6450afb/738662d6-6c41-4f3e-a588-8d054add7828"
+					(reference "U4")
+					(unit 1)
+				)
