File: pcb/Minicopter.kicad_pcb (KiCad board)
At the start: 2 copper layers, 136.1 x 135.4 mm, 57 parts, among them J1 USB_C_Receptacle_USB2.0_16P, J2 Conn_01x02, J3 Conn_01x02_Socket, J4 Conn_01x02_Socket, J5 Conn_01x02_Socket, J6 Conn_01x02_Socket, Q1 AO3401A, SW1 SS-12D00, T1 IRLML6344TRPBF, T2 IRLML6344TRPBF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

Commit message: fixed usb placement
Parts:
- moved J1 6.53 mm to (146.8, 129.3)
Routing:
- net GND: track 408.5 -> 580.1 mm
- net Net-(J1-CC1): track 2.92 -> 36.1 mm, vias 0 -> 2
- net Net-(J1-D+-PadA6): track 34.2 -> 12.1 mm
- net +BATT: track 431.1 -> 436.1 mm
- net Net-(J1-D--PadA7): track 11.9 -> 15.7 mm, vias 2 -> 4
- net Net-(J1-CC2): track 16.0 -> 18.1 mm
- net VBUS: track 102.4 -> 102.0 mm, vias 6 -> 7
